Commit message: Added fake CaseyControl, Working sim

File: snake/urdfFiles/snake.urdf (robot description, URDF)
Before this commit: robot snake, 8 links, 7 joints
Links:
- added link joint3
- added link link4; visual cylinder length=0.4 radius=.1
Joints:
- added joint joint3p: type continuous, parent link3, child joint3, origin xyz=.5 0 0 rpy=-1.57 0 0, axis 0 0 1
- added joint joint3y: type continuous, parent joint3, child link4, origin xyz=0 0 0 rpy=1.57 0 0, axis 0 0 1

Commit message: added max angle checkers, more tidying

File: snake/urdfFiles/snake.urdf (robot description, URDF)
Before this commit: robot snake, 10 links, 9 joints
Links:
- link imu1: geometry visual box size=0.005 0.005 0.005
- link imu2position: geometry visual box size=0.005 0.005 0.005
- link imu3: geometry visual box size=0.005 0.005 0.005
- link link1: geometry visual mesh filename=package://snake/urdfFiles/mesh/LinkStart.dae scale=0.001 0.001 0.001
- link link2: geometry visual mesh filename=package://snake/urdfFiles/mesh/LinkBothEnds.dae scale=0.001 0.001 0.001
- link link3: geometry visual mesh filename=package://snake/urdfFiles/mesh/LinkBothEnds.dae scale=0.001 0.001 0.001
- link link4: geometry visual mesh filename=package://snake/urdfFiles/mesh/LinkEnd.dae scale=0.001 0.001 0.001
Joints:
- joint imu1placement: origin xyz=0.25 0 0 -> xyz=0.1715 0 0
- joint imu2placement: origin xyz=0.25 0 0 -> xyz=0.1715 0 0
- joint imu3placement: origin xyz=0.25 0 0 -> xyz=0.1715 0 0
- joint joint1p: origin xyz=.5 0 0 rpy=-1.57 0 0 -> xyz=.2605 0 0 rpy=-1.57 0 0
- joint joint2p: origin xyz=.5 0 0 rpy=-1.57 0 0 -> xyz=.333 0 0 rpy=-1.57 0 0
- joint joint3p: origin xyz=.5 0 0 rpy=-1.57 0 0 -> xyz=.333 0 0 rpy=-1.57 0 0
